Commit message: Gazebo controls success

File: description/gazebo_control.xacro (robot description, xacro)
@@ -1,22 +1,42 @@
-<gazebo>
-  <plugin name="diff_drive" filename="libgazebo_ros_diff_drive.so">
-    <!-- Wheel Joints -->
-    <left_front_joint>left_front_joint</left_front_joint>
-    <right_front_joint>right_front_joint</right_front_joint>
-    <left_rear_joint>left_rear_joint</left_rear_joint>
-    <right_rear_joint>right_rear_joint</right_rear_joint>
-    <!-- Physical properties -->
-    <wheel_separation>0.44</wheel_separation> <!-- match y offsets of wheels -->
-    <wheel_diameter>0.1</wheel_diameter>
-    <max_wheel_torque>200</max_wheel_torque>
-    <max_wheel_acceleration>10.0</max_wheel_acceleration>
-    <!-- ROS Integration -->
-    <command_topic>/cmd_vel</command_topic>
-    <odometry_topic>odom</odometry_topic>
-    <odometry_frame>odom</odometry_frame>
-    <robot_base_frame>base_link</robot_base_frame>
-    <publish_odom>true</publish_odom>
-    <publish_odom_tf>true</publish_odom_tf>
-    <publish_wheel_tf>true</publish_wheel_tf>
-  </plugin>
-</gazebo>
+<?xml version="1.0"?>
+<robot xmlns:xacro="http://www.ros.org/wiki/xacro">
+    <gazebo>
+        <plugin name="skid_steer_drive" filename="libgazebo_ros_diff_drive.so">
+            <!-- Wheel Information -->
+            <num_wheel_pairs>2</num_wheel_pairs>
+            <left_joint>left_front_joint</left_joint>
+            <right_joint>right_front_joint</right_joint>
+            <left_joint>left_rear_joint</left_joint>
+            <right_joint>right_rear_joint</right_joint>
+            <wheel_separation>0.44</wheel_separation>
+            <wheel_diameter>0.1</wheel_diameter>
+            <!-- Limits -->
+            <max_wheel_torque>500</max_wheel_torque>
+            <max_wheel_acceleration>10.0</max_wheel_acceleration>
+            <ros>
+                <namespace>/</namespace>
+                <remapping>/cmd_vel:=cmd_vel</remapping>
+                <remapping>/odom:=odom</remapping>
+            </ros>
+            <!-- Output -->
+            <update_rate>30.0</update_rate>
+            <odometry_frame>odom</odometry_frame>
+            <robot_base_frame>base_link</robot_base_frame>
+            <publish_odom>true</publish_odom>
+            <publish_odom_tf>true</publish_odom_tf>
+            <publish_wheel_tf>true</publish_wheel_tf>
+            <odometry_topic>odom</odometry_topic>
+            <!-- <robot_base_frame>base_footprint</robot_base_frame> -->
+        </plugin>
+    <plugin name="rover_joint_state" filename="libgazebo_ros_joint_state_publisher.so">
+      <ros>
+          <remapping>~/out:=joint_states</remapping>
+      </ros>
+      <update_rate>30</update_rate>
+      <joint_name>left_front_joint</joint_name>
+      <joint_name>right_front_joint</joint_name>
+      <joint_name>left_rear_joint</joint_name>
+      <joint_name>right_rear_joint</joint_name>
+    </plugin>
+    </gazebo>
+</robot>

File: description/robot_core.xacro (robot description, xacro)
@@ -39,4 +39,7 @@
     </xacro:box_inertia>
   </link>
+  <gazebo reference="chassis">
+      <material>Gazebo/White</material>
+  </gazebo>
   <!--LEFT FRONT WHEEL JOINT-->
   <joint name="left_front_joint" type="continuous">
@@ -50,5 +53,5 @@
     <visual>
       <geometry>
-        <cylinder radius="0.05" length="0.04"/>
+        <cylinder radius="0.075" length="0.04"/>
       </geometry>
       <material name = "blue"/>
@@ -56,11 +59,14 @@
     <collision>
       <geometry>
-        <cylinder radius="0.05" length="0.04"/>
+        <cylinder radius="0.075" length="0.04"/>
       </geometry>
     </collision>
-    <xacro:cylinder_inertia mass="0.1" length="0.04" radius="0.05">
+    <xacro:cylinder_inertia mass="0.1" length="0.04" radius="0.075">
       <origin xyz="0.0 0.0 0.0" rpy="0.0 0.0 0.0"/>
     </xacro:cylinder_inertia>
   </link>
+  <gazebo reference="left_front">
+      <material>Gazebo/Blue</material>
+  </gazebo>
   <!--RIGHT FRONT WHEEL JOINT-->
   <joint name="right_front_joint" type="continuous">
@@ -74,5 +80,5 @@
     <visual>
       <geometry>
-        <cylinder radius="0.05" length="0.04"/>
+        <cylinder radius="0.075" length="0.04"/>
       </geometry>
       <material name = "blue"/>
@@ -80,11 +86,14 @@
     <collision>
       <geometry>
-        <cylinder radius="0.05" length="0.04"/>
+        <cylinder radius="0.075" length="0.04"/>
       </geometry>
     </collision>
-    <xacro:cylinder_inertia mass="0.1" length="0.04" radius="0.05">
+    <xacro:cylinder_inertia mass="0.1" length="0.04" radius="0.075">
       <origin xyz="0.0 0.0 0.0" rpy="0.0 0.0 0.0"/>
     </xacro:cylinder_inertia>
   </link>
+  <gazebo reference="right_front">
+      <material>Gazebo/Blue</material>
+  </gazebo>
   <!--LEFT REAR WHEEL JOINT-->
   <joint name="left_rear_joint" type="continuous">
@@ -98,5 +107,5 @@
     <visual>
       <geometry>
-        <cylinder radius="0.05" length="0.04"/>
+        <cylinder radius="0.075" length="0.04"/>
       </geometry>
       <material name = "blue"/>
@@ -104,11 +113,14 @@
     <collision>
       <geometry>
-        <cylinder radius="0.05" length="0.04"/>
+        <cylinder radius="0.075" length="0.04"/>
       </geometry>
     </collision>
-    <xacro:cylinder_inertia mass="0.1" length="0.04" radius="0.05">
+    <xacro:cylinder_inertia mass="0.1" length="0.04" radius="0.075">
       <origin xyz="0.0 0.0 0.0" rpy="0.0 0.0 0.0"/>
     </xacro:cylinder_inertia>
   </link>
+  <gazebo reference="left_rear">
+      <material>Gazebo/Blue</material>
+  </gazebo>
   <!--RIGHT REAR WHEEL JOINT-->
   <joint name="right_rear_joint" type="continuous">
@@ -122,5 +134,5 @@
     <visual>
       <geometry>
-        <cylinder radius="0.05" length="0.04"/>
+        <cylinder radius="0.075" length="0.04"/>
       </geometry>
       <material name = "blue"/>
@@ -128,10 +140,13 @@
     <collision>
       <geometry>
-        <cylinder radius="0.05" length="0.04"/>
+        <cylinder radius="0.075" length="0.04"/>
       </geometry>
     </collision>
-    <xacro:cylinder_inertia mass="0.1" length="0.04" radius="0.05">
+    <xacro:cylinder_inertia mass="0.1" length="0.04" radius="0.075">
       <origin xyz="0.0 0.0 0.0" rpy="0.0 0.0 0.0"/>
     </xacro:cylinder_inertia>
   </link>
+  <gazebo reference="right_rear">
+      <material>Gazebo/Blue</material>
+  </gazebo>
 </robot>
